Commit message: the result for learing process Creator Robot course

File: src/export5_URDF/urdf/keep_leg_export.urdf (robot description, URDF)
Before this commit: robot keep_leg_export, 19 links, 18 joints
Links:
- removed link base_footprint
- added link base_inertia, mass 1.0
- link base_link: mass 1.38302095240476 -> None; geometry collision mesh filename=package://keep_leg_export/meshes/base_link.STL scale=0.001 0.001 0.001; visual mesh filename=package://keep_leg_export/meshes/base_link.STL scale=1 1 1
Joints:
- removed joint base_joint
- added joint base_link_to_base_inertia: type fixed, parent base_link, child base_inertia, origin xyz=0 0 0 rpy=0 0 0
